Commit message: trabajo postparcial

File: src/description/odin_description.urdf (robot description, URDF)
Before this commit: robot odin, 2 links, 1 joints
Links:
- added link ultrasonic_front
- added link ultrasonic_left
- added link ultrasonic_right
- link base_link: geometry collision cylinder length=${base_height} radius=${base_radius}; visual cylinder length=${base_height} radius=${base_radius}
Joints:
- added joint ultrasonic_front_joint: type fixed, parent base_link, child ultrasonic_front, origin xyz=0.1 0 0 rpy=0 0 0
- added joint ultrasonic_left_joint: type fixed, parent base_link, child ultrasonic_left, origin xyz=0.0707 0.0707 0 rpy=0 0 0.7854
- added joint ultrasonic_right_joint: type fixed, parent base_link, child ultrasonic_right, origin xyz=0.0707 -0.0707 0 rpy=0 0 -0.7854
